Commit message: Update turtlebot_materials.urdf.xacro
removed comment in urdf file that made gazebo crash

File: gki_turtlebot_description/urdf/turtlebot_materials.urdf.xacro (robot description, xacro)
@@ -25,8 +25,3 @@
 		<color rgba="1.0 0.5 0.0 1.0"/>
 	</material>
-<!--
-	<material name="Caster">
-		<texture filename="package://pr2_ogre/Media/materials/textures/pr2_caster_texture.png" />
-	</material>
--->
 </robot>
