Commit message: added robot specific launch files for all our turtlebots

File: gki_turtlebot_description/robots/kobuki_hexagons_freiburg_kinect.urdf.xacro (robot description, xacro)
@@ -19,3 +19,7 @@
     <origin xyz="-0.04 0.0 0.008" rpy="0 0 0"/>
   </xacro:hokuyo_urg>
+  <xacro:include filename="$(find gki_sensors_description)/urdf/sick_rfu620.urdf.xacro" />
+  <xacro:sick_rfu620 name="rfid_sensor" parent="base_link" ros_topic="rfid_data">
+    <origin xyz="0.0 0.0 0.0" rpy="3.142 -0.785 0"/>
+  </xacro:sick_rfu620>
 </robot>
